Commit message: update my_robot_description pkg

File: my_robot_description/urdf/my_robot.urdf (robot description, URDF)
Before this commit: robot my_robot, 7 links, 6 joints
Links:
- removed link U_1
- removed link V_1
- removed link W_1
- removed link X_1
- removed link Y_1
- removed link Z_1
- added link base_footprint
- added link caster_wheel_link; visual sphere radius=0.05
- added link left_wheel_link; visual cylinder length=0.05 radius=0.1
- added link right_wheel_link; visual cylinder length=0.05 radius=0.1
- link base_link: mass 7.210677442504244 -> None; geometry visual box size=0.6 0.4 0.2
Joints:
- removed joint Rev28
- removed joint Rev29
- removed joint Rev30
- removed joint Rev31
- removed joint Rev32
- removed joint Rev33
- added joint base_caster_wheel_joint: type fixed, parent base_link, child caster_wheel_link, origin xyz=0.2 0 -0.05 rpy=0 0 0
- added joint base_joint: type fixed, parent base_footprint, child base_link, origin xyz=0 0 0.1 rpy=0 0 0
- added joint base_left_wheel_joint: type continuous, parent base_link, child left_wheel_link, origin xyz=-0.15 0.225 0 rpy=0 0 0, axis 0 1 0
- added joint base_right_wheel_joint: type continuous, parent base_link, child right_wheel_link, origin xyz=-0.15 -0.225 0 rpy=0 0 0, axis 0 1 0
