Commit message: added xacro

File: arm_robot_description/urdf/arm_robot.urdf.xacro (robot description, xacro)
@@ -1,4 +1,4 @@
 <?xml version="1.0" ?>
-<robot name="arm_robot">
+<robot name="arm_robot" xmlns:xacro="https://www.ros.org/wiki/xacro">
 <material name="silver">
   <color rgba="0.700 0.700 0.700 1.000"/>

File: my_robot_description/urdf/my_robot.urdf.xacro (robot description, xacro)
@@ -1,4 +1,9 @@
 <?xml version="1.0"?>
-<robot name="my_robot">
+<robot name="my_robot" xmlns:xacro="http://www.ros.org/wiki/xacro">
+    <xacro:property name="base_length" value="0.6" />
+    <xacro:property name="base_width" value="0.4" />
+    <xacro:property name="base_height" value="0.2" />
+    <xacro:property name="wheel_radius" value="0.1" />
+    <xacro:property name="wheel_length" value="0.05" />
     <material name="blue">
         <color rgba="0 0 0.5 1" />
@@ -11,7 +16,7 @@
         <visual>
             <geometry>
-                <box size="0.6 0.4 0.2" />
+                <box size="${base_length} ${base_width} ${base_height}" />
             </geometry>
-            <origin xyz="0 0 0.1" rpy="0 0 0" />
+            <origin xyz="0 0 ${base_height/2.0}" rpy="0 0 0" />
             <material name="blue" />
         </visual>
@@ -20,7 +25,7 @@
         <visual>
             <geometry>
-                <cylinder radius="0.1" length="0.05" />
+                <cylinder radius="${wheel_radius}" length="${wheel_length}" />
             </geometry>
-            <origin xyz="0 0 0" rpy="1.57 0 0" />
+            <origin xyz="0 0 0" rpy="${pi/2.0} 0 0" />
             <material name="grey" />
         </visual>
@@ -29,5 +34,5 @@
         <visual>
             <geometry>
-                <cylinder radius="0.1" length="0.05" />
+                <cylinder radius="${wheel_radius}" length="${wheel_length}" />
             </geometry>
             <origin xyz="0 0 0" rpy="1.57 0 0" />
@@ -47,10 +52,10 @@
         <parent link="base_footprint" />
         <child link="base_link" />
-        <origin xyz="0 0 0.1" rpy="0 0 0" />
+        <origin xyz="0 0 ${wheel_radius}" rpy="0 0 0" />
     </joint>
     <joint name="base_right_wheel_joint" type="continuous">
         <parent link="base_link" />
         <child link="right_wheel_link" />
-        <origin xyz="-0.15 -0.225 0" rpy="0 0 0" />
+        <origin xyz="${-base_length/4.0} -0.225 0" rpy="0 0 0" />
         <axis xyz="0 1 0" />
     </joint>
@@ -58,5 +63,5 @@
         <parent link="base_link" />
         <child link="left_wheel_link" />
-        <origin xyz="-0.15 0.225 0" rpy="0 0 0" />
+        <origin xyz="${-base_length/4.0} 0.225 0" rpy="0 0 0" />
         <axis xyz="0 1 0" />
     </joint>
@@ -64,5 +69,5 @@
         <parent link="base_link" />
         <child link="caster_wheel_link" />
-        <origin xyz="0.2 0 -0.05" rpy="0 0 0" />
+        <origin xyz="${base_length/3.0} 0 -0.05" rpy="0 0 0" />
     </joint>
 </robot>

Commit message: updates

File: arm_robot_description/urdf/arm_robot.urdf.xacro (robot description, xacro)
@@ -1,7 +1,6 @@
 <?xml version="1.0" ?>
 <robot name="arm_robot" xmlns:xacro="https://www.ros.org/wiki/xacro">
-<material name="silver">
-  <color rgba="0.700 0.700 0.700 1.000"/>
-</material>
+<xacro:include filename="$(find arm_robot_description)/urdf/materials.xacro" />
+<xacro:include filename="$(find arm_robot_description)/urdf/ruxonros2.gazebo" />
 <link name="base_link">
   <inertial>
@@ -13,5 +12,5 @@
     <origin xyz="0 0 0" rpy="0 0 0"/>
     <geometry>
-      <mesh filename="package://arm_robot_description/meshes/base_link.stl" scale="0.001 0.001 0.001"/>
+      <mesh filename="$(find arm_robot_description)/meshes/base_link.stl" scale="0.001 0.001 0.001"/>
     </geometry>
     <material name="silver"/>
@@ -20,5 +19,5 @@
     <origin xyz="0 0 0" rpy="0 0 0"/>
     <geometry>
-      <mesh filename="package://arm_robot_description/meshes/base_link.stl" scale="0.001 0.001 0.001"/>
+      <mesh filename="$(find arm_robot_description)/meshes/base_link.stl" scale="0.001 0.001 0.001"/>
     </geometry>
   </collision>
@@ -33,5 +32,5 @@
     <origin xyz="-0.0 -0.023029 -0.111" rpy="0 0 0"/>
     <geometry>
-      <mesh filename="package://arm_robot_description/meshes/X_1.stl" scale="0.001 0.001 0.001"/>
+      <mesh filename="$(find arm_robot_description)/meshes/X_1.stl" scale="0.001 0.001 0.001"/>
     </geometry>
     <material name="silver"/>
@@ -40,5 +39,5 @@
     <origin xyz="-0.0 -0.023029 -0.111" rpy="0 0 0"/>
     <geometry>
-      <mesh filename="package://arm_robot_description/meshes/X_1.stl" scale="0.001 0.001 0.001"/>
+      <mesh filename="$(find arm_robot_description)/meshes/X_1.stl" scale="0.001 0.001 0.001"/>
     </geometry>
   </collision>
@@ -53,5 +52,5 @@
     <origin xyz="-0.05713 -0.002855 -0.28806" rpy="0 0 0"/>
     <geometry>
-      <mesh filename="package://arm_robot_description/meshes/Y_1.stl" scale="0.001 0.001 0.001"/>
+      <mesh filename="$(find arm_robot_description)/meshes/Y_1.stl" scale="0.001 0.001 0.001"/>
     </geometry>
     <material name="silver"/>
@@ -60,5 +59,5 @@
     <origin xyz="-0.05713 -0.002855 -0.28806" rpy="0 0 0"/>
     <geometry>
-      <mesh filename="package://arm_robot_description/meshes/Y_1.stl" scale="0.001 0.001 0.001"/>
+      <mesh filename="$(find arm_robot_description)/meshes/Y_1.stl" scale="0.001 0.001 0.001"/>
     </geometry>
   </collision>
@@ -73,5 +72,5 @@
     <origin xyz="-0.04339 -0.003782 -0.548929" rpy="0 0 0"/>
     <geometry>
-      <mesh filename="package://arm_robot_description/meshes/Z_1.stl" scale="0.001 0.001 0.001"/>
+      <mesh filename="$(find arm_robot_description)/meshes/Z_1.stl" scale="0.001 0.001 0.001"/>
     </geometry>
     <material name="silver"/>
@@ -80,5 +79,5 @@
     <origin xyz="-0.04339 -0.003782 -0.548929" rpy="0 0 0"/>
     <geometry>
-      <mesh filename="package://arm_robot_description/meshes/Z_1.stl" scale="0.001 0.001 0.001"/>
+      <mesh filename="$(find arm_robot_description)/meshes/Z_1.stl" scale="0.001 0.001 0.001"/>
     </geometry>
   </collision>
@@ -93,5 +92,5 @@
     <origin xyz="0.000819 0.119908 -0.570126" rpy="0 0 0"/>
     <geometry>
-      <mesh filename="package://arm_robot_description/meshes/U_1.stl" scale="0.001 0.001 0.001"/>
+      <mesh filename="$(find arm_robot_description)/meshes/U_1.stl" scale="0.001 0.001 0.001"/>
     </geometry>
     <material name="silver"/>
@@ -100,5 +99,5 @@
     <origin xyz="0.000819 0.119908 -0.570126" rpy="0 0 0"/>
     <geometry>
-      <mesh filename="package://arm_robot_description/meshes/U_1.stl" scale="0.001 0.001 0.001"/>
+      <mesh filename="$(find arm_robot_description)/meshes/U_1.stl" scale="0.001 0.001 0.001"/>
     </geometry>
   </collision>
@@ -113,5 +112,5 @@
     <origin xyz="0.04021 0.254971 -0.568148" rpy="0 0 0"/>
     <geometry>
-      <mesh filename="package://arm_robot_description/meshes/V_1.stl" scale="0.001 0.001 0.001"/>
+      <mesh filename="$(find arm_robot_description)/meshes/V_1.stl" scale="0.001 0.001 0.001"/>
     </geometry>
     <material name="silver"/>
@@ -120,5 +119,5 @@
     <origin xyz="0.04021 0.254971 -0.568148" rpy="0 0 0"/>
     <geometry>
-      <mesh filename="package://arm_robot_description/meshes/V_1.stl" scale="0.001 0.001 0.001"/>
+      <mesh filename="$(find arm_robot_description)/meshes/V_1.stl" scale="0.001 0.001 0.001"/>
     </geometry>
   </collision>
@@ -133,5 +132,5 @@
     <origin xyz="0.00071 0.313516 -0.568205" rpy="0 0 0"/>
     <geometry>
-      <mesh filename="package://arm_robot_description/meshes/W_1.stl" scale="0.001 0.001 0.001"/>
+      <mesh filename="$(find arm_robot_description)/meshes/W_1.stl" scale="0.001 0.001 0.001"/>
     </geometry>
     <material name="silver"/>
@@ -140,5 +139,5 @@
     <origin xyz="0.00071 0.313516 -0.568205" rpy="0 0 0"/>
     <geometry>
-      <mesh filename="package://arm_robot_description/meshes/W_1.stl" scale="0.001 0.001 0.001"/>
+      <mesh filename="$(find arm_robot_description)/meshes/W_1.stl" scale="0.001 0.001 0.001"/>
     </geometry>
   </collision>
